File: AudioInjector.Octo.balanced.kicad_pcb (KiCad board)
At the start: 2 copper layers, 192.8 x 76.2 mm, 248 parts, among them K1 ck-6.35, K10 ck-6.35, K11 ck-6.35, K12 ck-6.35, K13 ck-6.35, K14 ck-6.35, K2 ck-6.35, K3 ck-6.35, K4 ck-6.35, K5 ck-6.35, K6 ck-6.35, K7 ck-6.35, K8 ck-6.35, K9 ck-6.35, P5 DAC_out, P6 ADC_in, T1 LFU9_8, T2 LFU9_8, T3 LFU9_8, T4 LFU9_8, U1 OP275, U10 OP275, U11 OP275, U12 OP275, U13 OP275, U14 OP275, U2 OP275, U3 OP275, U4 OP275, U5 OP275, U6 OP275, U7 OP275, U8 OP275, U9 OP275

Commit message: V1.6 of the balanced breakout for the Audioinjector Octo sound card for the Pi.
Parts:
- removed R109, R110, R111, R112, R113, R114, R115, R116, R117, R118, R119, R120, R121, R122, R123, R124: 47k, Resistors_SMD:R_0603
- removed T1, T2, T3, T4: LFU9_8, Common_Choke:LFU9.8
- added REF**: 1pin, Connect:1pin, F.Cu at (60.5, 93.5)
- added REF**: 1pin, Connect:1pin, F.Cu at (245.5, 93.5)
- added REF**: 1pin, Connect:1pin, F.Cu at (245.5, 102.5)
- added REF**: 1pin, Connect:1pin, F.Cu at (109.5, 102.5)
- C1, C10, C13, C14, C15, C16, C19, C2, C20, C21, C22, C25, C26, C27, C28, C31, C32, C33, C34, C37, C38, C39, C4, C40, C43, C44, C45, C46, C5, C7, C8, C9: value 1n -> ECHU1H102GX5
- C51, C52, C55, C56, C59, C60, C63, C64, C67, C68, C71, C72: value 470p -> ECHU1H471GX5
- L1, L2, L3, L4: value 47uH -> NLCV32T-470K
- P5, P6: moved to B.Cu
- R100, R101, R102, R103, R104, R49, R50, R51, R52, R53, R54, R59, R60, R61, R62, R63, R64, R69, R70, R71, R72, R73, R74, R79, R80, R81, R82, R83, R84, R89, R90, R91, R92, R93, R94, R99: value 390k -> 47k
- U1, U10, U11, U12, U13, U14, U2, U3, U4, U5, U6, U7, U8, U9: value OP275 -> NE5532
- moved R47 29.2 mm to (77.5, 76.2), turned to 0 degrees
- moved R35 29.1 mm to (125.5, 76.2), turned to 0 degrees
- moved R29 29.0 mm to (149.5, 76.2), turned to 0 degrees
- moved R6 29.0 mm to (245.5, 76.2), turned to 0 degrees
- moved R17 28.9 mm to (197.5, 76.2), turned to 0 degrees
- moved R23 28.9 mm to (173.5, 76.2), turned to 0 degrees
- moved R11 28.9 mm to (221.5, 76.2), turned to 0 degrees
- moved R41 28.8 mm to (101.5, 76.2), turned to 0 degrees
- moved R48 28.3 mm to (77.5, 73.8)
- moved R36 28.3 mm to (125.5, 73.8)
- moved R3 28.1 mm to (245.5, 73.8)
- moved R30 28.1 mm to (149.5, 73.8)
- moved R12 28.0 mm to (221.5, 73.8)
- moved R18 28.0 mm to (197.5, 73.8)
- moved R24 27.9 mm to (173.5, 73.8)
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Connections:
- net /Codec/5Va1 renamed /5Va1
- net /Codec/5Va2 renamed /5Va2
- net /Codec/5Vd1 renamed /5Vd1
- net /Codec/5Vd2 renamed /5Vd2
- net /Codec/In1+ renamed /In1+
- net /Codec/In1- renamed /In1-
- net /Codec/In2+ renamed /In2+
- net /Codec/In2- renamed /In2-
- net /Codec/In3+ renamed /In3+
- net /Codec/In3- renamed /In3-
- net /Codec/In4+ renamed /In4+
- net /Codec/In4- renamed /In4-
- net /Codec/In5+ renamed /In5+
- net /Codec/In5- renamed /In5-
- net /Codec/In6+ renamed /In6+
- net /Codec/In6- renamed /In6-
- net /Codec/OUT1+ renamed /OUT1+
- net /Codec/OUT1- renamed /OUT1-
- net /Codec/OUT2+ renamed /OUT2+
- net /Codec/OUT2- renamed /OUT2-
- net /Codec/OUT3+ renamed /OUT3+
- net /Codec/OUT3- renamed /OUT3-
- net /Codec/OUT4+ renamed /OUT4+
- net /Codec/OUT4- renamed /OUT4-
- net /Codec/OUT5+ renamed /OUT5+
- net /Codec/OUT5- renamed /OUT5-
- net /Codec/OUT6+ renamed /OUT6+
- net /Codec/OUT6- renamed /OUT6-
- net /Codec/OUT7+ renamed /OUT7+
- net /Codec/OUT7- renamed /OUT7-
- net /Codec/OUT8+ renamed /OUT8+
- net /Codec/OUT8- renamed /OUT8-
- net /Codec/V4++ renamed /V4++
- net /Codec/V4-+ renamed /V4-+
- net /Codec/V4Div+ renamed /V4Div+
- net /Codec/V4Div- renamed /V4Div-
- net /Codec/fb1+ renamed /fb1+
- net /Codec/fb1- renamed /fb1-
- net /Codec/fb2+ renamed /fb2+
- net /Codec/fb2- renamed /fb2-
- net /Codec/fb3+ renamed /fb3+
- net /Codec/fb3- renamed /fb3-
- net /Codec/fb4+ renamed /fb4+
- net /Codec/fb4- renamed /fb4-
- net /Codec/fb5+ renamed /fb5+
- net /Codec/fb5- renamed /fb5-
- net /Codec/fb6+ renamed /fb6+
- net /Codec/fb6- renamed /fb6-
- net /Codec/fb7+ renamed /fb7+
- net /Codec/fb7- renamed /fb7-
- net /Codec/fb8+ renamed /fb8+
- net /Codec/fb8- renamed /fb8-
- C1 pad 1: /Codec/AGND -> /AGNDD
- C13 pad 1: /Codec/AGND -> /AGNDD
- C14 pad 1: /Codec/AGND -> /AGNDD
- C19 pad 1: /Codec/AGND -> /AGNDD
- C20 pad 1: /Codec/AGND -> /AGNDD
- C25 pad 1: /Codec/AGND -> /AGNDD
- C26 pad 1: /Codec/AGND -> /AGNDD
- C31 pad 1: /Codec/AGND -> /AGNDD
- C32 pad 1: /Codec/AGND -> /AGNDD
- C37 pad 1: /Codec/AGND -> /AGNDD
- C38 pad 1: /Codec/AGND -> /AGNDD
- C4 pad 1: /Codec/AGND -> /AGNDD
- C43 pad 1: /Codec/AGND -> /AGNDD
- C44 pad 1: /Codec/AGND -> /AGNDD
- C7 pad 1: /Codec/AGND -> /AGNDD
- C73 pad 2: /Codec/AGND -> /AGNDA
- C74 pad 2: /Codec/AGND -> /AGNDA
- C75 pad 2: /Codec/AGND -> /AGNDD
- C76 pad 2: /Codec/AGND -> /AGNDD
- C77 pad 2: /Codec/AGND -> /AGNDD
- C78 pad 2: /Codec/AGND -> /AGNDD
- C79 pad 2: /Codec/AGND -> /AGNDD
- C8 pad 1: /Codec/AGND -> /AGNDD
- C80 pad 2: /Codec/AGND -> /AGNDD
- C81 pad 2: /Codec/AGND -> /AGNDD
- C82 pad 2: /Codec/AGND -> /AGNDD
- C83 pad 2: /Codec/AGND -> /AGNDA
- C84 pad 2: /Codec/AGND -> /AGNDA
- C85 pad 2: /Codec/AGND -> /AGNDA
- C86 pad 2: /Codec/AGND -> /AGNDA
- K1 pad 3: /Codec/AGND -> /AGNDD
- K10 pad 3: /Codec/AGND -> /AGNDA
- K11 pad 3: /Codec/AGND -> /AGNDA
- K12 pad 3: /Codec/AGND -> /AGNDA
- K13 pad 3: /Codec/AGND -> /AGNDA
- K14 pad 3: /Codec/AGND -> /AGNDA
- K2 pad 3: /Codec/AGND -> /AGNDD
- K3 pad 3: /Codec/AGND -> /AGNDD
- K4 pad 3: /Codec/AGND -> /AGNDD
- K5 pad 3: /Codec/AGND -> /AGNDD
- K6 pad 3: /Codec/AGND -> /AGNDD
- K7 pad 3: /Codec/AGND -> /AGNDD
- K8 pad 3: /Codec/AGND -> /AGNDD
- K9 pad 3: /Codec/AGND -> /AGNDA
- L1 pad 1: /Codec/5Vd1_ -> V5d
- L2 pad 1: /Codec/5Va1_ -> V5a
- L3 pad 1: /Codec/5Va2_ -> V5a
- L4 pad 1: /Codec/5Vd2_ -> V5d
- P5 pad 1: V5 -> V5d
- P5 pad 10: /Codec/AOUT5+ -> /AOUT6-
- P5 pad 11: /Codec/AOUT6+ -> /AOUT5-
- P5 pad 12: /Codec/AOUT5- -> /AOUT6+
- P5 pad 13: /Codec/AOUT4- -> /AOUT3+
- P5 pad 14: /Codec/AOUT3+ -> /AOUT4-
- P5 pad 15: /Codec/AOUT4+ -> /AOUT3-
- P5 pad 16: /Codec/AOUT3- -> /AOUT4+
- P5 pad 17: /Codec/AOUT2- -> /AOUT1+
- P5 pad 18: /Codec/AOUT1+ -> /AOUT2-
- P5 pad 19: /Codec/AOUT2+ -> /AOUT1-
- P5 pad 2: V5 -> V5d
- P5 pad 20: /Codec/AOUT1- -> /AOUT2+
- P5 pad 21: GNDA -> /AGNDD
- P5 pad 22: (no net) -> /AGNDD
- P5 pad 23: V5 -> V5d
- P5 pad 24: V5 -> V5d
- P5 pad 3: (no net) -> /AGNDD
- P5 pad 4: GNDA -> (no net)
- P5 pad 5: /Codec/AOUT8- -> /AOUT7+
- P5 pad 6: /Codec/AOUT7+ -> /AOUT8-
- P5 pad 7: /Codec/AOUT8+ -> /AOUT7-
- P5 pad 8: /Codec/AOUT7- -> /AOUT8+
- P5 pad 9: /Codec/AOUT6- -> /AOUT5+
- P6 pad 1: /Codec/ADC_fb1- -> V5a
- P6 pad 10: GNDA -> /ADC_fb3-
- P6 pad 11: /Codec/ADC_fb3+ -> /AGNDA
- P6 pad 12: GNDA -> /ADC_fb3+
- P6 pad 13: /Codec/ADC_fb4- -> /AGNDA
- P6 pad 14: GNDA -> /ADC_fb4-
- P6 pad 15: /Codec/ADC_fb4+ -> /AGNDA
- P6 pad 16: GNDA -> /ADC_fb4+
- P6 pad 17: /Codec/ADC_fb5- -> /AGNDA
- P6 pad 18: GNDA -> /ADC_fb5-
- P6 pad 19: /Codec/ADC_fb5+ -> /AGNDA
- P6 pad 2: V5 -> /ADC_fb1-
- P6 pad 20: GNDA -> /ADC_fb5+
- P6 pad 21: /Codec/ADC_fb6- -> V5a
- P6 pad 22: V5 -> /ADC_fb6-
- P6 pad 23: /Codec/ADC_fb6+ -> V5a
- P6 pad 24: V5 -> /ADC_fb6+
- P6 pad 3: /Codec/ADC_fb1+ -> V5a
- P6 pad 4: V5 -> /ADC_fb1+
- P6 pad 5: /Codec/ADC_fb2- -> /AGNDA
- P6 pad 6: GNDA -> /ADC_fb2-
- P6 pad 7: /Codec/ADC_fb2+ -> /AGNDA
- P6 pad 8: GNDA -> /ADC_fb2+
- P6 pad 9: /Codec/ADC_fb3- -> /AGNDA
- R1 pad 2: /Codec/AOUT1- -> /AOUT1-
- R100 pad 2: /Codec/AGND -> /AGNDA
- R102 pad 2: /Codec/AGND -> /AGNDA
- R104 pad 2: /Codec/AGND -> /AGNDA
- R105 pad 2: /Codec/ADC_fb6+ -> /ADC_fb6+
- R106 pad 2: /Codec/ADC_fb6- -> /ADC_fb6-
- R107 pad 2: /Codec/ADC_fb6+ -> /ADC_fb6+
- R108 pad 2: /Codec/ADC_fb6- -> /ADC_fb6-
- R11 pad 1: /Codec/AGND -> /AGNDD
- R12 pad 1: /Codec/AGND -> /AGNDD
- R13 pad 2: /Codec/AOUT3+ -> /AOUT3+
- R14 pad 2: /Codec/AOUT3- -> /AOUT3-
- R17 pad 1: /Codec/AGND -> /AGNDD
- R18 pad 1: /Codec/AGND -> /AGNDD
- R19 pad 2: /Codec/AOUT4+ -> /AOUT4+
- R20 pad 2: /Codec/AOUT4- -> /AOUT4-
- R23 pad 1: /Codec/AGND -> /AGNDD
- R24 pad 1: /Codec/AGND -> /AGNDD
- R25 pad 2: /Codec/AOUT5+ -> /AOUT5+
- R26 pad 2: /Codec/AOUT5- -> /AOUT5-
- R29 pad 1: /Codec/AGND -> /AGNDD
- R3 pad 1: /Codec/AGND -> /AGNDD
- R30 pad 1: /Codec/AGND -> /AGNDD
- R31 pad 2: /Codec/AOUT6+ -> /AOUT6+
- R32 pad 2: /Codec/AOUT6- -> /AOUT6-
- R35 pad 1: /Codec/AGND -> /AGNDD
- R36 pad 1: /Codec/AGND -> /AGNDD
- R37 pad 2: /Codec/AOUT7+ -> /AOUT7+
- R38 pad 2: /Codec/AOUT7- -> /AOUT7-
- R4 pad 2: /Codec/AOUT1+ -> /AOUT1+
- R41 pad 1: /Codec/AGND -> /AGNDD
- R42 pad 1: /Codec/AGND -> /AGNDD
- R43 pad 2: /Codec/AOUT8+ -> /AOUT8+
- R44 pad 2: /Codec/AOUT8- -> /AOUT8-
- R47 pad 1: /Codec/AGND -> /AGNDD
- R48 pad 1: /Codec/AGND -> /AGNDD
- R49 pad 2: /Codec/AGND -> /AGNDA
- R50 pad 2: /Codec/AGND -> /AGNDA
- R52 pad 2: /Codec/AGND -> /AGNDA
- R54 pad 2: /Codec/AGND -> /AGNDA
- R55 pad 2: /Codec/ADC_fb1+ -> /ADC_fb1+
- R56 pad 2: /Codec/ADC_fb1- -> /ADC_fb1-
- R57 pad 2: /Codec/ADC_fb1+ -> /ADC_fb1+
- R58 pad 2: /Codec/ADC_fb1- -> /ADC_fb1-
- R59 pad 2: /Codec/AGND -> /AGNDA
- R6 pad 1: /Codec/AGND -> /AGNDD
- R60 pad 2: /Codec/AGND -> /AGNDA
- R62 pad 2: /Codec/AGND -> /AGNDA
- R64 pad 2: /Codec/AGND -> /AGNDA
- R65 pad 2: /Codec/ADC_fb2+ -> /ADC_fb2+
- R66 pad 2: /Codec/ADC_fb2- -> /ADC_fb2-
- R67 pad 2: /Codec/ADC_fb2+ -> /ADC_fb2+
- R68 pad 2: /Codec/ADC_fb2- -> /ADC_fb2-
- R69 pad 2: /Codec/AGND -> /AGNDA
- R7 pad 2: /Codec/AOUT2+ -> /AOUT2+
- R70 pad 2: /Codec/AGND -> /AGNDA
- R72 pad 2: /Codec/AGND -> /AGNDA
- R74 pad 2: /Codec/AGND -> /AGNDA
- R75 pad 2: /Codec/ADC_fb3+ -> /ADC_fb3+
- R76 pad 2: /Codec/ADC_fb3- -> /ADC_fb3-
- R77 pad 2: /Codec/ADC_fb3+ -> /ADC_fb3+
- R78 pad 2: /Codec/ADC_fb3- -> /ADC_fb3-
- R79 pad 2: /Codec/AGND -> /AGNDA
- R8 pad 2: /Codec/AOUT2- -> /AOUT2-
- R80 pad 2: /Codec/AGND -> /AGNDA
- R82 pad 2: /Codec/AGND -> /AGNDA
- R84 pad 2: /Codec/AGND -> /AGNDA
- R85 pad 2: /Codec/ADC_fb4+ -> /ADC_fb4+
- R86 pad 2: /Codec/ADC_fb4- -> /ADC_fb4-
- R87 pad 2: /Codec/ADC_fb4+ -> /ADC_fb4+
- R88 pad 2: /Codec/ADC_fb4- -> /ADC_fb4-
- R89 pad 2: /Codec/AGND -> /AGNDA
- R90 pad 2: /Codec/AGND -> /AGNDA
- R92 pad 2: /Codec/AGND -> /AGNDA
- R94 pad 2: /Codec/AGND -> /AGNDA
- R95 pad 2: /Codec/ADC_fb5+ -> /ADC_fb5+
- R96 pad 2: /Codec/ADC_fb5- -> /ADC_fb5-
- R97 pad 2: /Codec/ADC_fb5+ -> /ADC_fb5+
- R98 pad 2: /Codec/ADC_fb5- -> /ADC_fb5-
- R99 pad 2: /Codec/AGND -> /AGNDA
- U1 pad 4: /Codec/AGND -> /AGNDD
- U10 pad 4: /Codec/AGND -> /AGNDA
- U11 pad 4: /Codec/AGND -> /AGNDA
- U12 pad 4: /Codec/AGND -> /AGNDA
- U13 pad 4: /Codec/AGND -> /AGNDA
- U14 pad 4: /Codec/AGND -> /AGNDA
- U2 pad 4: /Codec/AGND -> /AGNDD
- U3 pad 4: /Codec/AGND -> /AGNDD
- U4 pad 4: /Codec/AGND -> /AGNDD
- U5 pad 4: /Codec/AGND -> /AGNDD
- U6 pad 4: /Codec/AGND -> /AGNDD
- U7 pad 4: /Codec/AGND -> /AGNDD
- U8 pad 4: /Codec/AGND -> /AGNDD
- U9 pad 4: /Codec/AGND -> /AGNDA
Routing:
- net /Codec/AGND: track 1774.5 -> 0.00 mm, vias 283 -> 0
- net /AGNDD: track 0.00 -> 1387.3 mm, vias 0 -> 227
- net /AGNDA: track 0.00 -> 639.7 mm, vias 0 -> 80
- net GNDA: track 120.1 -> 0.00 mm
- net V5a: track 0.00 -> 97.1 mm
- net /AOUT1+: track 0.00 -> 92.9 mm
- net /Codec/AOUT1+: track 92.9 -> 0.00 mm
- net /Codec/AOUT1-: track 91.9 -> 0.00 mm
- net /AOUT1-: track 0.00 -> 91.9 mm
- net /Codec/AOUT8+: track 88.9 -> 0.00 mm
- net /AOUT8+: track 0.00 -> 88.9 mm
- net /AOUT8-: track 0.00 -> 88.9 mm
- net /Codec/AOUT8-: track 88.9 -> 0.00 mm
- net /Codec/AOUT7-: track 62.4 -> 0.00 mm
- net /AOUT7-: track 0.00 -> 62.4 mm
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- added copper zone on B.Cu, net /AGNDA
- added copper zone on F.Cu, net /AGNDA
- added copper zone on B.Cu, net /AGNDD
- added copper zone on F.Cu, net /AGNDD
- removed copper zone on B.Cu, net /Codec/AGND
- removed copper zone on F.Cu, net /Codec/AGND
Other:
- board size 192.8 x 76.2 mm -> 192.9 x 71.2 mm
- net class power_med added: clearance 0.2, trace_width 1.5, via_dia 0.6, via_drill 0.4
- board text added: "AudioInjector.net Octo Sound Card"
- board text added: "Balanced Breakout"
- board text added: "Flatmax (C) PPI8 in V1.6"
- board text added: "Flatmax (C) PPI8 out V1.6"
- board text removed: "Flatmax (C) PPI8 in V1.3"
- board text removed: "Flatmax (C) PPI8 out V1.3"
