File: AudioInjector.Octo.balanced.sch (KiCad schematic (older format))
At the start: 248 parts, among them K1 ck-6.35, K10 ck-6.35, K11 ck-6.35, K12 ck-6.35, K13 ck-6.35, K14 ck-6.35, K2 ck-6.35, K3 ck-6.35, K4 ck-6.35, K5 ck-6.35, K6 ck-6.35, K7 ck-6.35, K8 ck-6.35, K9 ck-6.35, P5 DAC_out, P6 ADC_in, T1 LFU9_8, T2 LFU9_8, T3 LFU9_8, T4 LFU9_8, U1 OP275, U10 OP275, U11 OP275, U12 OP275, U13 OP275, U14 OP275, U2 OP275, U3 OP275, U4 OP275, U5 OP275, U6 OP275, U7 OP275, U8 OP275, U9 OP275

Commit message: V1.6 of the balanced breakout for the Audioinjector Octo sound card for the Pi.
Parts:
- removed R109, R110, R111, R112, R113, R114, R115, R116, R117, R118, R119, R120, R121, R122, R123, R124: 47k, Resistors_SMD:R_0603, symbol R
- removed T1, T2, T3, T4: LFU9_8, Common_Choke:LFU9.8, symbol LFU9_8
- C1, C10, C13, C14, C15, C16, C19, C2, C20, C21, C22, C25, C26, C27, C28, C31, C32, C33, C34, C37, C38, C39, C4, C40, C43, C44, C45, C46, C5, C7, C8, C9: value 1n -> ECHU1H102GX5
- C51, C52, C55, C56, C59, C60, C63, C64, C67, C68, C71, C72: value 470p -> ECHU1H471GX5
- L1, L2, L3, L4: value 47uH -> NLCV32T-470K
- R100, R101, R102, R103, R104, R49, R50, R51, R52, R53, R54, R59, R60, R61, R62, R63, R64, R69, R70, R71, R72, R73, R74, R79, R80, R81, R82, R83, R84, R89, R90, R91, R92, R93, R94, R99: value 390k -> 47k
- U1, U10, U11, U12, U13, U14, U2, U3, U4, U5, U6, U7, U8, U9: value OP275 -> NE5532
Connections:
- net 5Va2_ is gone; now on net V5a: L3.1
- net 5Vd2_ is gone; now on net V5d: L4.1
- net ADC_fb1+: now also P6.4 (P4); no longer P6.3 (P3)
- net ADC_fb1-: now also P6.2 (P2); no longer P6.1 (P1)
- net ADC_fb2+: now also P6.8 (P8); no longer P6.7 (P7)
- net ADC_fb2-: now also P6.6 (P6); no longer P6.5 (P5)
- net ADC_fb3+: now also P6.12 (P12); no longer P6.11 (P11)
- net ADC_fb3-: now also P6.10 (P10); no longer P6.9 (P9)
- net ADC_fb4+: now also P6.16 (P16); no longer P6.15 (P15)
- net ADC_fb4-: now also P6.14 (P14); no longer P6.13 (P13)
- net ADC_fb5+: now also P6.20 (P20); no longer P6.19 (P19)
- net ADC_fb5-: now also P6.18 (P18); no longer P6.17 (P17)
- net ADC_fb6+: now also P6.24 (P24); no longer P6.23 (P23)
- net ADC_fb6-: now also P6.22 (P22); no longer P6.21 (P21)
- net AOUT1+: now also P5.17 (P17); no longer P5.18 (P18)
- net AOUT1-: now also P5.19 (P19); no longer P5.20 (P20)
- net AOUT2+: now also P5.20 (P20); no longer P5.19 (P19)
- net AOUT2-: now also P5.18 (P18); no longer P5.17 (P17)
- net AOUT3+: now also P5.13 (P13); no longer P5.14 (P14)
- net AOUT3-: now also P5.15 (P15); no longer P5.16 (P16)
- net AOUT4+: now also P5.16 (P16); no longer P5.15 (P15)
- net AOUT4-: now also P5.14 (P14); no longer P5.13 (P13)
- net AOUT5+: now also P5.9 (P9); no longer P5.10 (P10)
- net AOUT5-: now also P5.11 (P11); no longer P5.12 (P12)
- net AOUT6+: now also P5.12 (P12); no longer P5.11 (P11)
- net AOUT6-: now also P5.10 (P10); no longer P5.9 (P9)
- net AOUT7+: now also P5.5 (P5); no longer P5.6 (P6)
- net AOUT7-: now also P5.7 (P7); no longer P5.8 (P8)
- net AOUT8+: now also P5.8 (P8); no longer P5.7 (P7)
- net AOUT8-: now also P5.6 (P6); no longer P5.5 (P5)
- net MUTEC: now also P5.4 (P4); no longer P5.3 (P3)
- net AGNDD: now reaches P5.22 (P22)
- net AGNDD: now also C1.1, C13.1, C14.1, C19.1, C20.1, C25.1, C26.1, C31.1, C32.1, C37.1, C38.1, C4.1, C43.1, C44.1, C7.1, C75.2, C76.2, C77.2, C78.2, C79.2, C8.1, C80.2, C81.2, C82.2, K1.3, K2.3, K3.3, K4.3, K5.3, K6.3, K7.3, K8.3, P5.21 (P21), P5.3 (P3), R11.1, R12.1, R17.1, R18.1, R23.1, R24.1, R29.1, R3.1, R30.1, R35.1, R36.1, R41.1, R42.1, R47.1, R48.1, R6.1, U1.4 (V-), U1.4 (V-), U2.4 (V-), U2.4 (V-), U3.4 (V-), U3.4 (V-), U4.4 (V-), U4.4 (V-), U5.4 (V-), U5.4 (V-), U6.4 (V-), U6.4 (V-), U7.4 (V-), U7.4 (V-), U8.4 (V-), U8.4 (V-)
- net 5Va1_ renamed V5a
- net V5a: now also P6.1 (P1), P6.21 (P21), P6.23 (P23), P6.3 (P3)
- net 5Vd1_ renamed V5d
- net V5d: now also P5.1 (P1), P5.2 (P2), P5.23 (P23), P5.24 (P24)
- removed net AGND: C1.1, C13.1, C14.1, C19.1, C20.1, C25.1, C26.1, C31.1, C32.1, C37.1, C38.1, C4.1, C43.1, C44.1, C7.1, C73.2, C74.2, C75.2, C76.2, C77.2, C78.2, C79.2, C8.1, C80.2, C81.2, C82.2, C83.2, C84.2, C85.2, C86.2, K1.3, K10.3, K11.3, K12.3, K13.3, K14.3, K2.3, K3.3, K4.3, K5.3, K6.3, K7.3, K8.3, K9.3, R100.2, R102.2, R104.2, R11.1, R12.1, R17.1, R18.1, R23.1, R24.1, R29.1, R3.1, R30.1, R35.1, R36.1, R41.1, R42.1, R47.1, R48.1, R49.2, R50.2, R52.2, R54.2, R59.2, R6.1, R60.2, R62.2, R64.2, R69.2, R70.2, R72.2, R74.2, R79.2, R80.2, R82.2, R84.2, R89.2, R90.2, R92.2, R94.2, R99.2, U1.4 (V-), U1.4 (V-), U10.4 (V-), U10.4 (V-), U11.4 (V-), U11.4 (V-), U12.4 (V-), U12.4 (V-), U13.4 (V-), U13.4 (V-), U14.4 (V-), U14.4 (V-), U2.4 (V-), U2.4 (V-), U3.4 (V-), U3.4 (V-), U4.4 (V-), U4.4 (V-), U5.4 (V-), U5.4 (V-), U6.4 (V-), U6.4 (V-), U7.4 (V-), U7.4 (V-), U8.4 (V-), U8.4 (V-), U9.4 (V-), U9.4 (V-)
- removed net GNDA: P5.21 (P21), P5.4 (P4), P6.10 (P10), P6.12 (P12), P6.14 (P14), P6.16 (P16), P6.18 (P18), P6.20 (P20), P6.6 (P6), P6.8 (P8)
- removed net V5: P5.1 (P1), P5.2 (P2), P5.23 (P23), P5.24 (P24), P6.2 (P2), P6.22 (P22), P6.24 (P24), P6.4 (P4)
- new net AGNDA: C73.2, C74.2, C83.2, C84.2, C85.2, C86.2, K10.3, K11.3, K12.3, K13.3, K14.3, K9.3, P6.11 (P11), P6.13 (P13), P6.15 (P15), P6.17 (P17), P6.19 (P19), P6.5 (P5), P6.7 (P7), P6.9 (P9), R100.2, R102.2, R104.2, R49.2, R50.2, R52.2, R54.2, R59.2, R60.2, R62.2, R64.2, R69.2, R70.2, R72.2, R74.2, R79.2, R80.2, R82.2, R84.2, R89.2, R90.2, R92.2, R94.2, R99.2, U10.4 (V-), U10.4 (V-), U11.4 (V-), U11.4 (V-), U12.4 (V-), U12.4 (V-), U13.4 (V-), U13.4 (V-), U14.4 (V-), U14.4 (V-), U9.4 (V-), U9.4 (V-)
Other:
- moved on the sheet: C1, C10, C11, C12, C13, C14, C15, C16, C17, C18, C19, C2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
